File: a500plus-chipram-expansion.kicad_pcb (KiCad board)
At the start: 2 copper layers, 41.2 x 51.8 mm, 11 parts, among them J1 Expansion Header, J2 EN, U1 XRAS(0) 512KB, U2 XRAS(1) 512KB

Commit message: v1.1
Parts:
- J1: value Expansion Header -> A500 MEM EXP
- J2: value EN -> Enable
Routing:
- net +5V: track 183.4 -> 184.3 mm
- net XRAS(0): track 47.9 -> 47.1 mm
Other:
- board text added: "2x20 2.54mm CONNECTOR THIS SIDE"
- board text added: "Archer v1.1 @markbaseggio"
- board text added: "MB Chip RAM Expansion"
- board text added: "https://github.com/blark/a500plus-chipram-expansion"
- board text removed: "Archer-A500-v1 blark"
- board text removed: "MB Chip Ram Expansion"

Commit message: v2.0
Parts:
- removed J2: Enable, Connector_PinHeader_2.54mm:PinHeader_1x02_P2.54mm_Horizontal
- added C7: 10uF, Capacitor_SMD:C_0805_2012Metric_Pad1.15x1.40mm_HandSolder, F.Cu at (84.0, 82.2)
- added R1: 10K, Resistor_SMD:R_0805_2012Metric_Pad1.15x1.40mm_HandSolder, F.Cu at (103.3, 37.0)
- added SW1: <ENABLE, Button_Switch_THT:SW_CuK_JS202011AQN_DPDT_Angled, F.Cu at (98.5, 37.8)
- C4, U2: moved to F.Cu
- moved C5 30.0 mm to (106.3, 40.5), turned to 0 degrees
- moved C3 20.9 mm to (87.9, 40.6), turned to 180 degrees
- moved C4 15.1 mm to (102.4, 40.5), turned to 0 degrees
- moved U2 10.5 mm to (97.0, 48.5), turned to 270 degrees
- moved C1 10.5 mm to (102.3, 60.5), turned to 0 degrees
- moved C6 9.97 mm to (87.8, 60.6)
- moved U1 9.51 mm to (97.0, 68.5), turned to 270 degrees
- moved C2 2.75 mm to (106.3, 60.5)
- moved REF** 1.46 mm to (105.2, 80.5)
Routing:
- net GND: track 14.5 -> 86.7 mm, vias 7 -> 10
- net +5V: track 184.3 -> 141.8 mm, vias 16 -> 7
- net /12: track 37.7 -> 71.6 mm, vias 1 -> 4
- net /1: track 51.6 -> 74.0 mm, vias 0 -> 2
- net /15: track 30.4 -> 51.6 mm, vias 1 -> 2
- net /2: track 45.8 -> 66.4 mm, vias 0 -> 2
- net /11: track 42.2 -> 60.7 mm, vias 1 -> 2
- net /0: track 51.8 -> 67.8 mm, vias 0 -> 2
- net /13: track 39.4 -> 54.2 mm, vias 1 -> 2
- net XWE: track 51.4 -> 37.5 mm, vias 4 -> 2
- net XCASL: track 40.9 -> 53.5 mm
- net /14: track 35.1 -> 46.6 mm, vias 1 -> 2
- net XRAS(1): track 28.2 -> 17.9 mm, vias 0 -> 1
- net XOE: track 41.6 -> 51.3 mm
- net /4: track 49.2 -> 58.9 mm, vias 0 -> 2
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- removed copper zone on F.Cu, net GND
Other:
- board text added: "1"
- board text added: "Archer v2.0 @markbaseggio"
- board text added: "THIS SIDE DOWN"
- board text removed: "Archer v1.1 @markbaseggio"
